Commit message: fixed urdf

File: arm_description/urdf/arm.urdf.xacro (robot description, xacro)
@@ -13,10 +13,10 @@
         <geometry>
             <mesh filename="package://arm_description/meshes/stand/mounting_plate.stl"/>
-        <\geometry>
+        </geometry>
         <material name="white">
-    <\visual>
+    </visual>
     <inertial>
         <origin xyz="0 0 0" rpy="0 0 0"/>
-    <\inertial>
-  <\link>
+    </inertial>
+  </link>
 </robot>
