Commit message: control sig

File: arm_description/control/arm.ros2_control.xacro (robot description, xacro)
@@ -1,46 +1,10 @@
 <?xml version="1.0"?>
 <robot xmlns:xacro="http://www.ros.org/wiki/xacro">
-  <xacro:macro name="fws_robot_ros2_control">
+  <xacro:macro name="arm_ros2_control">
     <ros2_control name="fws" type="system">
       <hardware>
           <plugin>gz_ros2_control/GazeboSimSystem</plugin>
       </hardware>
-      <joint name="fl_wheel_joint">
-        <command_interface name="velocity">
-          <param name="min">-1</param>
-          <param name="max">1</param>
-        </command_interface>
-        <state_interface name="position"/>
-        <state_interface name="velocity"/>
-        <state_interface name="effort"/>
-      </joint>
-      <joint name="fr_wheel_joint">
-        <command_interface name="velocity">
-          <param name="min">-1</param>
-          <param name="max">1</param>
-        </command_interface>
-        <state_interface name="position"/>
-        <state_interface name="velocity"/>
-        <state_interface name="effort"/>
-      </joint>
-      <joint name="rl_wheel_joint">
-        <command_interface name="velocity">
-          <param name="min">-1</param>
-          <param name="max">1</param>
-        </command_interface>
-        <state_interface name="position"/>
-        <state_interface name="velocity"/>
-        <state_interface name="effort"/>
-      </joint>
-      <joint name="rr_wheel_joint">
-        <command_interface name="velocity">
-          <param name="min">-1</param>
-          <param name="max">1</param>
-        </command_interface>
-        <state_interface name="position"/>
-        <state_interface name="velocity"/>
-        <state_interface name="effort"/>
-      </joint>
-      <joint name="fl_steering_joint">
+      <joint name="J1">
         <command_interface name="position">
           <param name="min">-3.14</param>
@@ -51,5 +15,5 @@
         <state_interface name="effort"/>
       </joint>
-      <joint name="fr_steering_joint">
+      <joint name="J2">
         <command_interface name="position">
           <param name="min">-3.14</param>
@@ -60,5 +24,5 @@
         <state_interface name="effort"/>
       </joint>
-      <joint name="rl_steering_joint">
+      <joint name="J3">
         <command_interface name="position">
           <param name="min">-3.14</param>
@@ -69,5 +33,14 @@
         <state_interface name="effort"/>
       </joint>
-      <joint name="rr_steering_joint">
+      <joint name="J4">
+        <command_interface name="position">
+          <param name="min">-3.14</param>
+          <param name="max">3.14</param>
+        </command_interface>
+        <state_interface name="position"/>
+        <state_interface name="velocity"/>
+        <state_interface name="effort"/>
+      </joint>
+      <joint name="J5">
         <command_interface name="position">
           <param name="min">-3.14</param>

File: arm_description/model/arm.urdf.xacro (robot description, xacro)
@@ -1,5 +1,5 @@
 <?xml version="1.0"?>
 <robot name="arm" xmlns:xacro="https://www.ros.org/wiki/xacro">
-        <xacro:include filename="$(find arm_description)/model/arm.gazebo"
+        <xacro:include filename="$(find arm_description)/control/arm.ros2_control.xacro" />
         <material name="white">
                 <color rgba="1 1 1 1" />
@@ -12,5 +12,5 @@
         </material>
         <!--LINKS-->
-        <link name="base_footprint"> </links>
+        <link name="base_footprint"> </link>
         <joint name="base_footprint_link" type="fixed">
                 <parent link="base_footprint"/>
@@ -275,69 +275,3 @@
                 <origin xyz="0 0 0.0078" rpy="0 0 0" />
         </joint>
-        <!--ROS2 Control-->
-        <ros2_control name="GazeboSystem" type="system">
-                <hardware>
-                        <plugin>gazebo_ros2_control_GazeboSystem</plugin>
-                </hardware>
-                <joint name="J1">
-                        <command_interface name="position">
-                                <param name="min">-3.14</param>
-                                <param name="max">3.14</param>
-                        </command_interface>
-                        <state_interface name="position">
-                                <param name="inital_value">0</param>
-                        </state_interface>
-                        <state_interface name="velocity">
-                        <state_interface name="effort">
-                </joint>
-                <joint name="J2">
-                        <command_interface name="position">
-                                <param name="min">-3.14</param>
-                                <param name="max">3.14</param>
-                        </command_interface>
-                        <state_interface name="position">
-                                <param name="inital_value">0</param>
-                        </state_interface>
-                        <state_interface name="velocity">
-                        <state_interface name="effort">
-                </joint>
-                <joint name="J3">
-                        <command_interface name="position">
-                                <param name="min">-3.14</param>
-                                <param name="max">3.14</param>
-                        </command_interface>
-                        <state_interface name="position">
-                                <param name="inital_value">0</param>
-                        </state_interface>
-                        <state_interface name="velocity">
-                        <state_interface name="effort">
-                </joint>
-                <joint name="J4">
-                        <command_interface name="position">
-                                <param name="min">-3.14</param>
-                                <param name="max">3.14</param>
-                        </command_interface>
-                        <state_interface name="position">
-                                <param name="inital_value">0</param>
-                        </state_interface>
-                        <state_interface name="velocity">
-                        <state_interface name="effort">
-                </joint>
-                <joint name="J5">
-                        <command_interface name="position">
-                                <param name="min">-3.14</param>
-                                <param name="max">3.14</param>
-                        </command_interface>
-                        <state_interface name="position">
-                                <param name="inital_value">0</param>
-                        </state_interface>
-                        <state_interface name="velocity">
-                        <state_interface name="effort">
-                </joint>
-        </ros2_control>
-        <gazebo>
-                <plugin filename="libgazebo_ros2_control.so" name="gazebo_ros2_control">
-                        <parameters>$(find arm_description)/config/joint_controller.yaml</parameters>
-                </plugin>
-        </gazebo>
 </robot>
