Commit message: added end effector model and updated ros2 controllers

File: arm_description/control/arm_ros2_control.xacro (robot description, xacro)
@@ -51,4 +51,31 @@
                 <state_interface name="effort"/>
             </joint>
+            <joint name="J6">
+                <command_interface name="position">
+                    <param name="min">-3.05</param>
+                    <param name="max">3.05</param>
+                </command_interface>
+                <state_interface name="position"/>
+                <state_interface name="velocity"/>
+                <state_interface name="effort"/>
+            </joint>
+            <joint name="JLeft">
+                <command_interface name="position">
+                    <param name="min">0</param>
+                    <param name="max">0.025</param>
+                </command_interface>
+                <state_interface name="position"/>
+                <state_interface name="velocity"/>
+                <state_interface name="effort"/>
+            </joint>
+            <joint name="JRight">
+                <command_interface name="position">
+                    <param name="min">0</param>
+                    <param name="max">0.025</param>
+                </command_interface>
+                <state_interface name="position"/>
+                <state_interface name="velocity"/>
+                <state_interface name="effort"/>
+            </joint>
         </ros2_control>
     </xacro:macro>

File: arm_description/model/arm.urdf (robot description, URDF)
Before this commit: robot arm, 18 links, 17 joints
Links:
- removed link base_pulley
- removed link base_structure
- removed link base_structure_cover
- removed link base_tube
- removed link baseplate
- removed link fore_pulley
- removed link fore_rotation
- removed link fore_structure
- removed link j5_bearing_adapter_1
- removed link j5_bearing_adapter_2
- removed link j6_housing
- removed link j6_nema8
- removed link upper_bearing_mount
- removed link upper_housing
- removed link upper_pulley
- removed link upper_structure
- removed link world
- added link ee, mass 0.027464; collision mesh filename=package://arm_description/model/meshes/ee.STL; visual mesh filename=package://arm_description/model/meshes/ee.STL
- added link fingerL, mass 0.0069323; collision mesh filename=package://arm_description/model/meshes/fingerL.STL; visual mesh filename=package://arm_description/model/meshes/fingerL.STL
- added link fingerR, mass 0.0069323; collision mesh filename=package://arm_description/model/meshes/fingerR.STL; visual mesh filename=package://arm_description/model/meshes/fingerR.STL
- added link link1, mass 0.35633; collision mesh filename=package://arm_description/model/meshes/link1.STL; visual mesh filename=package://arm_description/model/meshes/link1.STL
- added link link2, mass 0.26746; collision mesh filename=package://arm_description/model/meshes/link2.STL; visual mesh filename=package://arm_description/model/meshes/link2.STL
- added link link3, mass 0.222311320377134; collision mesh filename=package://arm_description/model/meshes/link3.STL; visual mesh filename=package://arm_description/model/meshes/link3.STL
- added link link4, mass 0.1696257012172; collision mesh filename=package://arm_description/model/meshes/link4.STL; visual mesh filename=package://arm_description/model/meshes/link4.STL
- added link link5, mass 0.0179895273320859; collision mesh filename=package://arm_description/model/meshes/link5.STL; visual mesh filename=package://arm_description/model/meshes/link5.STL
- link base_link: mass 1 -> 0.43666; geometry collision mesh filename=package://arm_description/model/meshes/base_link.STL; visual mesh filename=package://arm_description/model/meshes/base_link.STL
Joints:
- removed joint base_pulley_structure_joint
- removed joint base_structure_cover_joint
- removed joint base_to_world
- removed joint end_housing_nema8
- removed joint fore_pully_structure_joint
- removed joint fore_rotation_bearing_1
- removed joint fore_rotation_bearing_2
- removed joint stand_link_tube_joint
- removed joint stand_tube_baseplate_joint
- removed joint upper_mount_housing
- removed joint upper_pulley_structure
- removed joint upper_structure_mount
- added joint J6: type continuous, parent link5, child ee, origin xyz=-0.0199666324199864 -0.0127552190119366 0.00382596102472059 rpy=-1.41021344284507 -0.0773897000977449 2.12675451737731, axis 0 0 1
- added joint JLeft: type prismatic, parent ee, child fingerL, origin xyz=-0.025364 -0.0020424 0.02375 rpy=-1.5708 0 -1.5708, axis 1 0 0, limit lower=0 upper=0 effort=0 velocity=0
- added joint JRight: type prismatic, parent ee, child fingerR, origin xyz=0.026636 0.0014336 0.02375 rpy=-1.8383 0 1.5708, axis 1 0 0, limit lower=0 upper=0 effort=0 velocity=0
- joint J1: axis 0 0 1 -> 0 1 0; child base_pulley -> link1; origin xyz=0 0 0.016 rpy=0 0 0 -> xyz=0.087103 -0.077154 0.054376 rpy=1.5708 0 -0.17957; parent baseplate -> base_link
- joint J2: axis 0 0 1 -> 0.178603115585449 0 0.983921199641095; child upper_pulley -> link2; limit lower=-0.349 upper=1.5708 effort=10 velocity=3 -> (none); origin xyz=0.037 -0.0337 0.04 rpy=1.5708 0 3.1415 -> xyz=-0.0383525749921799 0.0583000000000001 -0.0013208705506468 rpy=0.0114835938093404 -0.000363602890144003 0.0633037833578822; parent base_structure -> link1; type revolute -> continuous
- joint J3: axis 0 0 1 -> 0.178603115585449 0 0.983921199641095; child fore_pulley -> link3; limit lower=-3.1415 upper=1.5708 effort=10 velocity=3 -> (none); origin xyz=0.0 0.16 0.0 rpy=0 0 1.5708 -> xyz=0.01012184118035 0.159668946677294 -0.00183733450496954 rpy=-0.0341579908525323 -0.00324248866976051 -0.189267104095329; parent upper_structure -> link2; type revolute -> continuous
- joint J4: axis 0 0 1 -> 0.97586466350816 0.127708020083281 -0.17714067890384; child fore_rotation -> link4; limit lower=-3.1415 upper=1.5708 effort=10 velocity=3 -> (none); origin xyz=0.015 0.035 0.0245 rpy=0 1.5708 1.5708 -> xyz=-3.63625649351731E-05 0.0148771771133325 0.0105252497783941 rpy=0.0192434154802188 0.00255235780533698 -0.00346944801670467; parent fore_structure -> link3; type revolute -> continuous
- joint J5: axis 1 0 0 -> 0.176090142676508 0.0195610841602276 0.98417967142115; child j6_housing -> link5; limit lower=-3.1415 upper=1.5708 effort=10 velocity=3 -> (none); origin xyz=0 0 0.0925 rpy=0 0 0 -> xyz=-0.135560517031385 -0.0176394821004389 0.0246051802150107 rpy=-3.01860336767631 0.324554663782284 0.719451490827395; parent j5_bearing_adapter_1 -> link4; type revolute -> continuous
