Commit message: added end effector model and updated ros2 controllers

File: arm_description/model/arm.urdf.xacro (robot description, xacro)
@@ -1,523 +1,482 @@
-<?xml version="1.0"?>
+<?xml version="1.0" encoding="utf-8"?>
+<!-- This URDF was automatically created by SolidWorks to URDF Exporter! Originally created by Stephen Brawner (brawner@gmail.com)
+     Commit Version: 1.6.0-4-g7f85cfe  Build Version: 1.6.7995.38578
+     For more information, please see http://wiki.ros.org/sw_urdf_exporter -->
+<!-- Hunter Ellis: modified to work with gazebo -->
 <robot xmlns:xacro="https://www.ros.org/wiki/xacro" name="arm">
-        <xacro:include filename="$(find arm_description)/model/arm.gazebo.xacro" />
-        <xacro:include filename="$(find arm_description)/control/arm_ros2_control.xacro" />
-        <xacro:arg name="add_world" default="true"/>
-        <xacro:arg name="base_link" default="base_link"/>
-        <xacro:arg name="base_type" default="g_shape"/>
-        <xacro:arg name="flange_link" default="base_link"/>
-        <xacro:arg name="use_camera" default="false"/>
-        <xacro:arg name="use_gazebo" default="false"/>
-        <xacro:arg name="use_gripper" default="true"/>
-        <material name="white">
-                <color rgba="1 1 1 1" />
-        </material>
-        <material name="grey">
-                <color rgba="0.5 0.5 0.5 1" />
-        </material>
-        <material name="red">
-                <color rgba="1 0 0 1" />
-        </material>
-        <link name="world"/>
-        <joint name="base_to_world" type="fixed">
-                <child link="base_link" />
-                <parent link="world" />
-                <origin xyz="0 0 0" rpy="0 0 0" />
-        </joint>
-        <!--stand-->
-        <link name="base_link">
-                <visual>
-                        <geometry>
-                                <mesh filename="package://arm_description/model/meshes/stand/mounting_plate.stl" scale ="0.001 0.001 0.001"/>
-                        </geometry>
-                        <origin xyz="0.06 -0.06 0" rpy="1.5708 0 3.1415" />
-                        <material name="white" />
-                </visual>
-                <collision>
-                        <geometry>
-                                <mesh filename="package://arm_description/model/meshes/stand/mounting_plate.dae" scale ="0.001 0.001 0.001"/>
-                        </geometry>
-                        <origin xyz="0.06 -0.06 0" rpy="1.5708 0 3.1415" />
-                        <material name="white" />
-                </collision>
-                <inertial>
-                        <origin xyz="0 0 0" />
-                        <mass value="1" />
-                        <inertia ixx="0.0001873" ixy="0" ixz="0" iyy="0.000055" iyz="0" izz="0.0002283" />
-                </inertial>
-        </link>
-        <link name="base_tube">
-                <visual>
-                        <geometry>
-                                <mesh filename="package://arm_description/model/meshes/stand/base_tube.stl" scale ="0.001 0.001 0.001"/>
-                        </geometry>
-                        <origin xyz="0.04 -0.04 0" rpy="1.5708 0 3.1415" />
-                        <material name="white" />
-                </visual>
-                <collision>
-                        <geometry>
-                                <mesh filename="package://arm_description/model/meshes/stand/base_tube.dae" scale ="0.001 0.001 0.001"/>
-                        </geometry>
-                        <origin xyz="0.04 -0.04 0" rpy="1.5708 0 3.1415" />
-                        <material name="white" />
-                </collision>
-                <inertial>
-                        <origin xyz="0 0 0" />
-                        <mass value="1" />
-                        <inertia ixx="0.0001873" ixy="0" ixz="0" iyy="0.000055" iyz="0" izz="0.0002283" />
-                </inertial>
-        </link>
-        <link name="baseplate">
-                <visual>
-                        <geometry>
-                                <mesh filename="package://arm_description/model/meshes/stand/baseplate.stl" scale ="0.001 0.001 0.001"/>
-                        </geometry>
-                        <origin xyz="0.04 -0.04 0" rpy="1.5708 0 3.1415" />
-                        <material name="white" />
-                </visual>
-                <collision>
-                        <geometry>
-                                <mesh filename="package://arm_description/model/meshes/stand/baseplate.dae" scale ="0.001 0.001 0.001"/>
-                        </geometry>
-                        <origin xyz="0.04 -0.04 0" rpy="1.5708 0 3.1415" />
-                        <material name="white" />
-                </collision>
-                <inertial>
-                        <origin xyz="0 0 0" />
-                        <mass value="1" />
-                        <inertia ixx="0.0001873" ixy="0" ixz="0" iyy="0.000055" iyz="0" izz="0.0002283" />
-                </inertial>
-        </link>
-        <!--base-->
-        <link name="base_pulley">
-                <visual>
-                        <geometry>
-                                <mesh filename="package://arm_description/model/meshes/base/base_pulley.stl" scale ="0.001 0.001 0.001"/>
-                        </geometry>
-                        <origin xyz="0.035 -0.035 0.009" rpy="1.5708 1.5708 3.1415" />
-                        <material name="white" />
-                </visual>
-                <collision>
-                        <geometry>
-                                <mesh filename="package://arm_description/model/meshes/base/base_pulley.dae" scale ="0.001 0.001 0.001"/>
-                        </geometry>
-                        <origin xyz="0.035 -0.035 0.009" rpy="1.5708 1.5708 3.1415" />
-                        <material name="white" />
-                </collision>
-                <inertial>
-                        <origin xyz="0 0 0" />
-                        <mass value="1" />
-                        <inertia ixx="0.0001873" ixy="0" ixz="0" iyy="0.000055" iyz="0" izz="0.0002283" />
-                </inertial>
-        </link>
-        <link name="base_structure">
-                <visual>
-                        <geometry>
-                                <mesh filename="package://arm_description/model/meshes/base/base_structure.stl" scale ="0.001 0.001 0.001"/>
-                        </geometry>
-                        <origin xyz="0.0774 0.035 0" rpy="1.5708 0 -1.5708" />
-                        <material name="white" />
-                </visual>
-                <collision>
-                        <geometry>
-                                <mesh filename="package://arm_description/model/meshes/base/base_structure.dae" scale ="0.001 0.001 0.001"/>
-                        </geometry>
-                        <origin xyz="0.0774 0.035 0" rpy="1.5708 0 -1.5708" />
-                        <material name="white" />
-                </collision>
-                <inertial>
-                        <origin xyz="0 0 0" />
-                        <mass value="1" />
-                        <inertia ixx="0.0001873" ixy="0" ixz="0" iyy="0.000055" iyz="0" izz="0.0002283" />
-                </inertial>
-        </link>
-        <link name="base_structure_cover">
-                <visual>
-                        <geometry>
-                                <mesh filename="package://arm_description/model/meshes/base/base_structure_cover.stl" scale ="0.001 0.001 0.001"/>
-                        </geometry>
-                        <origin xyz="-0.0826 -0.02 0" rpy="1.5708 0 0" />
-                        <material name="white" />
-                </visual>
-                <collision>
-                        <geometry>
-                                <mesh filename="package://arm_description/model/meshes/base/base_structure_cover.dae" scale ="0.001 0.001 0.001"/>
-                        </geometry>
-                        <origin xyz="-0.0826 -0.02 0" rpy="1.5708 0 0" />
-                        <material name="white" />
-                </collision>
-                <inertial>
-                        <origin xyz="0 0 0" />
-                        <mass value="1" />
-                        <inertia ixx="0.0001873" ixy="0" ixz="0" iyy="0.000055" iyz="0" izz="0.0002283" />
-                </inertial>
-        </link>
-        <!--upperarm-->
-        <link name="upper_pulley">
-                <visual>
-                        <geometry>
-                                <mesh filename="package://arm_description/model/meshes/upperarm/j2_pulley.stl" scale ="0.001 0.001 0.001"/>
-                        </geometry>
-                        <origin xyz="-0.04 -0.04 0" rpy="0 0 0" />
-                        <material name="white" />
-                </visual>
-                <collision>
-                        <geometry>
-                                <mesh filename="package://arm_description/model/meshes/upperarm/j2_pulley.dae" scale ="0.001 0.001 0.001"/>
-                        </geometry>
-                        <origin xyz="-0.04 -0.04 0" rpy="0 0 0" />
-                        <material name="white" />
-                </collision>
-                <inertial>
-                        <origin xyz="0 0 0" />
-                        <mass value="1" />
-                        <inertia ixx="0.0001873" ixy="0" ixz="0" iyy="0.000055" iyz="0" izz="0.0002283" />
-                </inertial>
-        </link>
-        <link name="upper_structure">
-                <visual>
-                        <geometry>
-                                <mesh filename="package://arm_description/model/meshes/upperarm/upper_structure.stl" scale ="0.001 0.001 0.001"/>
-                        </geometry>
-                        <origin xyz="0.042 -0.03 0" rpy="0 3.1415 0" />
-                        <material name="white" />
-                </visual>
-                <collision>
-                        <geometry>
-                                <mesh filename="package://arm_description/model/meshes/upperarm/upper_structure.dae" scale ="0.001 0.001 0.001"/>
-                        </geometry>
-                        <origin xyz="0.042 -0.03 0" rpy="0 3.1415 0" />
-                        <material name="white" />
-                </collision>
-                <inertial>
-                        <origin xyz="0 0 0" />
-                        <mass value="1" />
-                        <inertia ixx="0.0001873" ixy="0" ixz="0" iyy="0.000055" iyz="0" izz="0.0002283" />
-                </inertial>
-        </link>
-        <link name="upper_bearing_mount">
-                <visual>
-                        <geometry>
-                                <mesh filename="package://arm_description/model/meshes/upperarm/upper_bearing_mount.stl" scale ="0.001 0.001 0.001"/>
-                        </geometry>
-                        <origin xyz="0.042 -0.03 -0.00025" rpy="0 3.1415 0" />
-                        <material name="white" />
-                </visual>
-                <collision>
-                        <geometry>
-                                <mesh filename="package://arm_description/model/meshes/upperarm/upper_bearing_mount.dae" scale ="0.001 0.001 0.001"/>
-                        </geometry>
-                        <origin xyz="0.042 -0.03 -0.00025" rpy="0 3.1415 0" />
-                        <material name="white" />
-                </collision>
-                <inertial>
-                        <origin xyz="0 0 0" />
-                        <mass value="1" />
-                        <inertia ixx="0.0001873" ixy="0" ixz="0" iyy="0.000055" iyz="0" izz="0.0002283" />
-                </inertial>
-        </link>
-        <link name="upper_housing">
-                <visual>
-                        <geometry>
-                                <mesh filename="package://arm_description/model/meshes/upperarm/upper_housing.stl" scale ="0.001 0.001 0.001"/>
-                        </geometry>
-                        <origin xyz="0.028 -0.03 -0.062" rpy="0 0 0" />
-                        <material name="white" />
-                </visual>
-                <collision>
-                        <geometry>
-                                <mesh filename="package://arm_description/model/meshes/upperarm/upper_housing.dae" scale ="0.001 0.001 0.001"/>
-                        </geometry>
-                        <origin xyz="0.028 -0.03 -0.062" rpy="0 0 0" />
-                        <material name="white" />
-                </collision>
-                <inertial>
-                        <origin xyz="0 0 0" />
-                        <mass value="1" />
-                        <inertia ixx="0.0001873" ixy="0" ixz="0" iyy="0.000055" iyz="0" izz="0.0002283" />
-                </inertial>
-        </link>
-        <!--forearm-->
-        <link name="fore_pulley">
-                <visual>
-                        <geometry>
-                                <mesh filename="package://arm_description/model/meshes/forearm/j3_pulley.stl" scale ="0.001 0.001 0.001"/>
-                        </geometry>
-                        <origin xyz="-0.035 -0.035 0.0175" rpy="0 1.5708 0" />
-                        <material name="white" />
-                </visual>
-                <collision>
-                        <geometry>
-                                <mesh filename="package://arm_description/model/meshes/forearm/j3_pulley.dae" scale ="0.001 0.001 0.001"/>
-                        </geometry>
-                        <origin xyz="-0.035 -0.035 0.0175" rpy="0 1.5708 0" />
-                        <material name="white" />
-                </collision>
-                <inertial>
-                        <origin xyz="0 0 0" />
-                        <mass value="1" />
-                        <inertia ixx="0.0001873" ixy="0" ixz="0" iyy="0.000055" iyz="0" izz="0.0002283" />
-                </inertial>
-        </link>
-        <link name="fore_structure">
-                <visual>
-                        <geometry>
-                                <mesh filename="package://arm_description/model/meshes/forearm/forearm_structure.stl" scale ="0.001 0.001 0.001"/>
-                        </geometry>
-                        <origin xyz="-0.045 -0.043 0" rpy="3.1415 -1.5708 1.5708" />
-                        <material name="white" />
-                </visual>
-                <collision>
-                        <geometry>
-                                <mesh filename="package://arm_description/model/meshes/forearm/forearm_structure.dae" scale ="0.001 0.001 0.001"/>
-                        </geometry>
-                        <origin xyz="-0.045 -0.043 0" rpy="3.1415 -1.5708 1.5708" />
-                        <material name="white" />
-                </collision>
-                <inertial>
-                        <origin xyz="0 0 0" />
-                        <mass value="1" />
-                        <inertia ixx="0.0001873" ixy="0" ixz="0" iyy="0.000055" iyz="0" izz="0.0002283" />
-                </inertial>
-        </link>
-        <link name="fore_rotation">
-                <visual>
-                        <geometry>
-                                <mesh filename="package://arm_description/model/meshes/forearm/forearm_rotation.stl" scale ="0.001 0.001 0.001"/>
-                        </geometry>
-                        <origin xyz="-0.033 -0.0175 0" rpy="0 0 0" />
-                        <material name="white" />
-                </visual>
-                <collision>
-                        <geometry>
-                                <mesh filename="package://arm_description/model/meshes/forearm/forearm_rotation.dae" scale ="0.001 0.001 0.001"/>
-                        </geometry>
-                        <origin xyz="-0.033 -0.0175 0" rpy="0 0 0" />
-                        <material name="white" />
-                </collision>
-                <inertial>
-                        <origin xyz="0 0 0" />
-                        <mass value="1" />
-                        <inertia ixx="0.0001873" ixy="0" ixz="0" iyy="0.000055" iyz="0" izz="0.0002283" />
-                </inertial>
-        </link>
-        <link name="j5_bearing_adapter_1">
-                <visual>
-                        <geometry>
-                                <mesh filename="package://arm_description/model/meshes/forearm/j5_bearing_adapter.stl" scale ="0.001 0.001 0.001"/>
-                        </geometry>
-                        <origin xyz="-0.023 0.011 0.10525" rpy="1.5708 1.5708 0" />
-                        <material name="white" />
-                </visual>
-                <collision>
-                        <geometry>
-                                <mesh filename="package://arm_description/model/meshes/forearm/j5_bearing_adapter.dae" scale ="0.001 0.001 0.001"/>
-                        </geometry>
-                        <origin xyz="-0.023 0.011 0.10525" rpy="1.5708 1.5708 0" />
-                        <material name="white" />
-                </collision>
-                <inertial>
-                        <origin xyz="0 0 0" />
-                        <mass value="1" />
-                        <inertia ixx="0.0001873" ixy="0" ixz="0" iyy="0.000055" iyz="0" izz="0.0002283" />
-                </inertial>
-        </link>
-        <link name="j5_bearing_adapter_2">
-                <visual>
-                        <geometry>
-                                <mesh filename="package://arm_description/model/meshes/forearm/j5_bearing_adapter.stl" scale ="0.001 0.001 0.001"/>
-                        </geometry>
-                        <origin xyz="0.023 -0.011 0.09525" rpy="-1.5708 1.5708 0" />
-                        <material name="white" />
-                </visual>
-                <collision>
-                        <geometry>
-                                <mesh filename="package://arm_description/model/meshes/forearm/j5_bearing_adapter.dae" scale ="0.001 0.001 0.001"/>
-                        </geometry>
-                        <origin xyz="0.023 -0.011 0.09525" rpy="-1.5708 1.5708 0" />
-                        <material name="white" />
-                </collision>
-                <inertial>
-                        <origin xyz="0 0 0" />
-                        <mass value="1" />
-                        <inertia ixx="0.0001873" ixy="0" ixz="0" iyy="0.000055" iyz="0" izz="0.0002283" />
-                </inertial>
-        </link>
-        <link name="j6_housing">
-                <visual>
-                        <geometry>
-                                <mesh filename="package://arm_description/model/meshes/forearm/j6_housing.stl" scale ="0.001 0.001 0.001"/>
-                        </geometry>
-                        <origin xyz="-0.01385 -0.01085 -0.02" rpy="0 0 0" />
-                        <material name="white" />
-                </visual>
-                <collision>
-                        <geometry>
-                                <mesh filename="package://arm_description/model/meshes/forearm/j6_housing.dae" scale ="0.001 0.001 0.001"/>
-                        </geometry>
-                        <origin xyz="-0.01385 -0.01085 -0.02" rpy="0 0 0" />
-                        <material name="white" />
-                </collision>
-                <inertial>
-                        <origin xyz="0 0 0" />
-                        <mass value="1" />
-                        <inertia ixx="0.0001873" ixy="0" ixz="0" iyy="0.000055" iyz="0" izz="0.0002283" />
-                </inertial>
-        </link>
-        <!--end effector-->
-        <link name="j6_nema8">
-                <visual>
-                        <geometry>
-                                <mesh filename="package://arm_description/model/meshes/forearm/j6_nema8.stl" scale ="0.001 0.001 0.001"/>
-                        </geometry>
-                        <origin xyz="0 0 0" rpy="0 0 0" />
-                        <material name="red" />
-                </visual>
-                <collision>
-                        <geometry>
-                                <mesh filename="package://arm_description/model/meshes/forearm/j6_nema8.dae" scale ="0.001 0.001 0.001"/>
-                        </geometry>
-                        <origin xyz="0 0 0" rpy="0 0 0" />
-                        <material name="red" />
-                </collision>
-                <inertial>
-                        <origin xyz="0 0 0" />
-                        <mass value="1" />
-                        <inertia ixx="0.0001873" ixy="0" ixz="0" iyy="0.000055" iyz="0" izz="0.0002283" />
-                </inertial>
-        </link>
-        <!--JOINTS-->
-        <!--stand joints-->
-        <joint name="stand_link_tube_joint" type="fixed">
-                <parent link="base_link" />
-                <child link="base_tube" />
-                <origin xyz="0 0 0.02" rpy="0 0 0" />
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
File: arm_description/model/camera/camera.xacro (robot description, xacro)
@@ -1,5 +1,5 @@
 <?xml version="1.0"?>
 <robot name="delirobo" xmlns:xacro="http://ros.org/wiki/xacro">
-  <xacro:include filename="$(find robot_description)/urdf/camera/camera.gazebo"/>
+  <xacro:include filename="$(find arm_description)/model/camera/camera.gazebo"/>
   <xacro:macro name="camera_v0" params="parent *joint_origin">
 	<joint name="camera_joint" type="fixed">
@@ -11,10 +11,10 @@
 	  <visual>
 		<geometry>
-		  <mesh filename="package://robot_description/meshes/visual/camera.dae"/>
+			<mesh filename="package://arm_description/model/meshes/camera/camera.dae"/>
 		</geometry>
 	  </visual>
 	  <collision>
 		<geometry>
-		  <mesh filename="package://robot_description/meshes/collision/camera.stl"/>
+			<mesh filename="package://arm_description/model/meshes/camera/camera.stl"/>
 		</geometry>
 	  </collision>
