Commit message: updated controllers and cv model

File: arm_description/control/arm_ros2_control.xacro (robot description, xacro)
@@ -63,5 +63,5 @@
                 <command_interface name="position">
                     <param name="min">0</param>
-                    <param name="max">0.025</param>
+                    <param name="max">1</param>
                 </command_interface>
                 <state_interface name="position"/>
@@ -72,5 +72,5 @@
                 <command_interface name="position">
                     <param name="min">0</param>
-                    <param name="max">0.025</param>
+                    <param name="max">1</param>
                 </command_interface>
                 <state_interface name="position"/>

File: arm_description/model/arm.urdf (robot description, URDF)
Before this commit: robot arm, 9 links, 8 joints
Joints:
- joint J1: limit (none) -> lower=-3.1415 upper=3.1415 effort=1 velocity=1; type continuous -> revolute

File: arm_description/model/arm.urdf.xacro (robot description, xacro)
@@ -10,5 +10,5 @@
   <xacro:include filename="$(find arm_description)/model/camera/camera.xacro"/>
   <xacro:camera_v0 parent="base_link">
-    <origin xyz="0 0 0.7" rpy="0 ${PI/2} 0"/>
+    <origin xyz="-0.1 0 0.7" rpy="0 ${PI/2} ${PI}"/>
   </xacro:camera_v0>
   <xacro:camera_gazebo_v0/>
@@ -20,5 +20,5 @@
     <child link="base_link" />
     <parent link="world" />
-    <origin xyz="0 0 0" rpy="0 0 0" />
+    <origin xyz="0.15 0 0" rpy="0 0 ${PI}" />
   </joint>
   <link
@@ -419,6 +419,6 @@
       lower="0"
       upper="0.025"
-      effort="0"
-      velocity="0" />
+      effort="10"
+      velocity="0.1" />
   </joint>
   <link
@@ -475,7 +475,21 @@
       lower="0"
       upper="0.025"
-      effort="0"
-      velocity="0" />
-  </joint>
+      effort="10"
+      velocity="0.1" />
+  </joint>
+  <gazebo reference="fingerL">
+    <mu1>1.0</mu1>
+    <mu2>1.0</mu2>
+    <kp>1000000.0</kp>
+    <kd>10.0</kd>
+    <material>Gazebo/White</material>
+  </gazebo>
+  <gazebo reference="fingerR">
+    <mu1>1.0</mu1>
+    <mu2>1.0</mu2>
+    <kp>1000000.0</kp>
+    <kd>10.0</kd>
+    <material>Gazebo/White</material>
+  </gazebo>
   <xacro:arm_gazebo/>
   <xacro:arm_ros2_control/>
