Commit message: gazebo integration

File: arm_description/model/arm.urdf.xacro (robot description, xacro)
@@ -1,4 +1,4 @@
 <?xml version="1.0"?>
-<robot name="arm" xmlns:xacro="https://www.ros.org/wiki/xacro">
+<robot xmlns:xacro="https://www.ros.org/wiki/xacro" name="arm">
         <xacro:include filename="$(find arm_description)/control/arm.ros2_control.xacro" />
         <material name="white">
@@ -11,9 +11,17 @@
                 <color rgba="1 0 0 1" />
         </material>
+        <link name="world"/>
+        <joint name="fix_world" type="fixed">
+                <parent link="world"/>
+                <child link="base_footprint"/>
+                <origin xyz="0 0 -0.055"/>
+        </joint>
         <!--LINKS-->
-        <link name="base_footprint"> </link>
+        <link name="base_footprint">
+        </link>
         <joint name="base_footprint_link" type="fixed">
                 <parent link="base_footprint"/>
                 <child link="base_link"/>
+                <origin xyz="0 0 0"/>
         </joint>
         <!--stand-->
@@ -22,8 +30,22 @@
                         <geometry>
                                 <mesh filename="package://arm_description/model/meshes/stand/mounting_plate.stl" scale ="0.001 0.001 0.001"/>
-                        </geometry>
                         <origin xyz="0.06 -0.06 0" rpy="1.5708 0 3.1415" />
                         <material name="white" />
-                </visual>
+                        </geometry>
+                        <origin xyz="0.06 -0.06 0" rpy="1.5708 0 3.1415" />
+                        <material name="white" />
+                </visual>
+                <collision>
+                        <geometry>
+                                <mesh filename="package://arm_description/model/meshes/stand/mounting_plate.dae" scale ="0.001 0.001 0.001"/>
+                        </geometry>
+                        <origin xyz="0.06 -0.06 0" rpy="1.5708 0 3.1415" />
+                        <material name="white" />
+                </collision>
+                <inertial>
+                        <origin xyz="0 0 0" />
+                        <mass value="1" />
+                        <inertia ixx="0.0001873" ixy="0" ixz="0" iyy="0.000055" iyz="0" izz="0.0002283" />
+                </inertial>
         </link>
         <link name="base_tube">
@@ -35,4 +57,16 @@
                         <material name="white" />
                 </visual>
+                <collision>
+                        <geometry>
+                                <mesh filename="package://arm_description/model/meshes/stand/base_tube.dae" scale ="0.001 0.001 0.001"/>
+                        </geometry>
+                        <origin xyz="0.04 -0.04 0" rpy="1.5708 0 3.1415" />
+                        <material name="white" />
+                </collision>
+                <inertial>
+                        <origin xyz="0 0 0" />
+                        <mass value="1" />
+                        <inertia ixx="0.0001873" ixy="0" ixz="0" iyy="0.000055" iyz="0" izz="0.0002283" />
+                </inertial>
         </link>
         <link name="baseplate">
@@ -44,4 +78,16 @@
                         <material name="white" />
                 </visual>
+                <collision>
+                        <geometry>
+                                <mesh filename="package://arm_description/model/meshes/stand/baseplate.dae" scale ="0.001 0.001 0.001"/>
+                        </geometry>
+                        <origin xyz="0.04 -0.04 0" rpy="1.5708 0 3.1415" />
+                        <material name="white" />
+                </collision>
+                <inertial>
+                        <origin xyz="0 0 0" />
+                        <mass value="1" />
+                        <inertia ixx="0.0001873" ixy="0" ixz="0" iyy="0.000055" iyz="0" izz="0.0002283" />
+                </inertial>
         </link>
         <!--base-->
@@ -54,4 +100,16 @@
                         <material name="white" />
                 </visual>
+                <collision>
+                        <geometry>
+                                <mesh filename="package://arm_description/model/meshes/base/base_pulley.dae" scale ="0.001 0.001 0.001"/>
+                        </geometry>
+                        <origin xyz="0.035 -0.035 0.009" rpy="1.5708 1.5708 3.1415" />
+                        <material name="white" />
+                </collision>
+                <inertial>
+                        <origin xyz="0 0 0" />
+                        <mass value="1" />
+                        <inertia ixx="0.0001873" ixy="0" ixz="0" iyy="0.000055" iyz="0" izz="0.0002283" />
+                </inertial>
         </link>
         <link name="base_structure">
@@ -63,4 +121,16 @@
                         <material name="white" />
                 </visual>
+                <collision>
+                        <geometry>
+                                <mesh filename="package://arm_description/model/meshes/base/base_structure.dae" scale ="0.001 0.001 0.001"/>
+                        </geometry>
+                        <origin xyz="0.0774 0.035 0" rpy="1.5708 0 -1.5708" />
+                        <material name="white" />
+                </collision>
+                <inertial>
+                        <origin xyz="0 0 0" />
+                        <mass value="1" />
+                        <inertia ixx="0.0001873" ixy="0" ixz="0" iyy="0.000055" iyz="0" izz="0.0002283" />
+                </inertial>
         </link>
         <link name="base_structure_cover">
@@ -72,4 +142,16 @@
                         <material name="white" />
                 </visual>
+                <collision>
+                        <geometry>
+                                <mesh filename="package://arm_description/model/meshes/base/base_structure_cover.dae" scale ="0.001 0.001 0.001"/>
+                        </geometry>
+                        <origin xyz="-0.0826 -0.02 0" rpy="1.5708 0 0" />
+                        <material name="white" />
+                </collision>
+                <inertial>
+                        <origin xyz="0 0 0" />
+                        <mass value="1" />
+                        <inertia ixx="0.0001873" ixy="0" ixz="0" iyy="0.000055" iyz="0" izz="0.0002283" />
+                </inertial>
         </link>
         <!--upperarm-->
@@ -82,4 +164,16 @@
                         <material name="white" />
                 </visual>
+                <collision>
+                        <geometry>
+                                <mesh filename="package://arm_description/model/meshes/upperarm/j2_pulley.dae" scale ="0.001 0.001 0.001"/>
+                        </geometry>
+                        <origin xyz="-0.04 -0.04 0" rpy="0 0 0" />
+                        <material name="white" />
+                </collision>
+                <inertial>
+                        <origin xyz="0 0 0" />
+                        <mass value="1" />
+                        <inertia ixx="0.0001873" ixy="0" ixz="0" iyy="0.000055" iyz="0" izz="0.0002283" />
+                </inertial>
         </link>
         <link name="upper_structure">
@@ -91,4 +185,16 @@
                         <material name="white" />
                 </visual>
+                <collision>
+                        <geometry>
+                                <mesh filename="package://arm_description/model/meshes/upperarm/upper_structure.dae" scale ="0.001 0.001 0.001"/>
+                        </geometry>
+                        <origin xyz="0.042 -0.03 0" rpy="0 3.1415 0" />
+                        <material name="white" />
+                </collision>
+                <inertial>
+                        <origin xyz="0 0 0" />
+                        <mass value="1" />
+                        <inertia ixx="0.0001873" ixy="0" ixz="0" iyy="0.000055" iyz="0" izz="0.0002283" />
+                </inertial>
         </link>
         <link name="upper_bearing_mount">
@@ -100,4 +206,16 @@
                         <material name="white" />
                 </visual>
+                <collision>
+                        <geometry>
+                                <mesh filename="package://arm_description/model/meshes/upperarm/upper_bearing_mount.dae" scale ="0.001 0.001 0.001"/>
+                        </geometry>
+                        <origin xyz="0.042 -0.03 -0.00025" rpy="0 3.1415 0" />
+                        <material name="white" />
+                </collision>
+                <inertial>
+                        <origin xyz="0 0 0" />
+                        <mass value="1" />
+                        <inertia ixx="0.0001873" ixy="0" ixz="0" iyy="0.000055" iyz="0" izz="0.0002283" />
+                </inertial>
         </link>
         <link name="upper_housing">
@@ -109,4 +227,16 @@
                         <material name="white" />
                 </visual>
+                <collision>
+                        <geometry>
+                                <mesh filename="package://arm_description/model/meshes/upperarm/upper_housing.dae" scale ="0.001 0.001 0.001"/>
+                        </geometry>
+                        <origin xyz="0.028 -0.03 -0.062" rpy="0 0 0" />
+                        <material name="white" />
+                </collision>
+                <inertial>
+                        <origin xyz="0 0 0" />
+                        <mass value="1" />
+                        <inertia ixx="0.0001873" ixy="0" ixz="0" iyy="0.000055" iyz="0" izz="0.0002283" />
+                </inertial>
         </link>
         <!--forearm-->
@@ -119,4 +249,16 @@
                         <material name="white" />
                 </visual>
+                <collision>
+                        <geometry>
+                                <mesh filename="package://arm_description/model/meshes/forearm/j3_pulley.dae" scale ="0.001 0.001 0.001"/>
+                        </geometry>
+                        <origin xyz="-0.035 -0.035 0.0175" rpy="0 1.5708 0" />
+                        <material name="white" />
+                </collision>
+                <inertial>
+                        <origin xyz="0 0 0" />
+                        <mass value="1" />
+                        <inertia ixx="0.0001873" ixy="0" ixz="0" iyy="0.000055" iyz="0" izz="0.0002283" />
+                </inertial>
         </link>
         <link name="fore_structure">
@@ -128,4 +270,16 @@
                         <material name="white" />
                 </visual>
+                <collision>
+                        <geometry>
+                                <mesh filename="package://arm_description/model/meshes/forearm/forearm_structure.dae" scale ="0.001 0.001 0.001"/>
+                        </geometry>
+                        <origin xyz="-0.045 -0.043 0" rpy="3.1415 -1.5708 1.5708" />
+                        <material name="white" />
+                </collision>
+                <inertial>
+                        <origin xyz="0 0 0" />
+                        <mass value="1" />
+                        <inertia ixx="0.0001873" ixy="0" ixz="0" iyy="0.000055" iyz="0" izz="0.0002283" />
+                </inertial>
         </link>
         <link name="fore_rotation">
@@ -137,4 +291,16 @@
                         <material name="white" />
                 </visual>
+                <collision>
+                        <geometry>
+                                <mesh filename="package://arm_description/model/meshes/forearm/forearm_rotation.dae" scale ="0.001 0.001 0.001"/>
+                        </geometry>
+                        <origin xyz="-0.033 -0.0175 0" rpy="0 0 0" />
+                        <material name="white" />
+                </collision>
+                <inertial>
+                        <origin xyz="0 0 0" />
+                        <mass value="1" />
+                        <inertia ixx="0.0001873" ixy="0" ixz="0" iyy="0.000055" iyz="0" izz="0.0002283" />
+                </inertial>
         </link>
         <link name="j5_bearing_adapter_1">
@@ -146,4 +312,16 @@
                         <material name="white" />
                 </visual>
+                <collision>
+                        <geometry>
+                                <mesh filename="package://arm_description/model/meshes/forearm/j5_bearing_adapter.dae" scale ="0.001 0.001 0.001"/>
+                        </geometry>
+                        <origin xyz="-0.023 0.011 0.10525" rpy="1.5708 1.5708 0" />
+                        <material name="white" />
+                </collision>
+                <inertial>
+                        <origin xyz="0 0 0" />
+                        <mass value="1" />
+                        <inertia ixx="0.0001873" ixy="0" ixz="0" iyy="0.000055" iyz="0" izz="0.0002283" />
+                </inertial>
         </link>
         <link name="j5_bearing_adapter_2">
@@ -155,4 +333,16 @@
                         <material name="white" />
                 </visual>
+                <collision>
+                        <geometry>
+                                <mesh filename="package://arm_description/model/meshes/forearm/j5_bearing_adapter.dae" scale ="0.001 0.001 0.001"/>
+                        </geometry>
+                        <origin xyz="0.023 -0.011 0.09525" rpy="-1.5708 1.5708 0" />
+                        <material name="white" />
+                </collision>
+                <inertial>
+                        <origin xyz="0 0 0" />
+                        <mass value="1" />
+                        <inertia ixx="0.0001873" ixy="0" ixz="0" iyy="0.000055" iyz="0" izz="0.0002283" />
+                </inertial>
         </link>
         <link name="j6_housing">
@@ -164,4 +354,16 @@
                         <material name="white" />
                 </visual>
+                <collision>
+                        <geometry>
+                                <mesh filename="package://arm_description/model/meshes/forearm/j6_housing.dae" scale ="0.001 0.001 0.001"/>
+                        </geometry>
+                        <origin xyz="-0.01385 -0.01085 -0.02" rpy="0 0 0" />
+                        <material name="white" />
+                </collision>
+                <inertial>
+                        <origin xyz="0 0 0" />
+                        <mass value="1" />
+                        <inertia ixx="0.0001873" ixy="0" ixz="0" iyy="0.000055" iyz="0" izz="0.0002283" />
+                </inertial>
         </link>
         <!--end effector-->
@@ -174,4 +376,16 @@
                         <material name="red" />
                 </visual>
+                <collision>
+                        <geometry>
+                                <mesh filename="package://arm_description/model/meshes/forearm/j6_nema8.dae" scale ="0.001 0.001 0.001"/>
+                        </geometry>
+                        <origin xyz="0 0 0" rpy="0 0 0" />
+                        <material name="red" />
+                </collision>
+                <inertial>
+                        <origin xyz="0 0 0" />
+                        <mass value="1" />
+                        <inertia ixx="0.0001873" ixy="0" ixz="0" iyy="0.000055" iyz="0" izz="0.0002283" />
+                </inertial>
         </link>
         <!--JOINTS-->

Commit message: fixed gz origin

File: arm_description/model/arm.urdf.xacro (robot description, xacro)
@@ -15,5 +15,5 @@
                 <parent link="world"/>
                 <child link="base_footprint"/>
-                <origin xyz="0 0 -0.055"/>
+                <origin xyz="0 0 0"/>
         </joint>
         <!--LINKS-->

Commit message: joint trajectory control node

File: arm_description/model/arm.urdf.xacro (robot description, xacro)
@@ -423,5 +423,5 @@
                 <child link="upper_pulley"/>
                 <origin xyz="0.037 -0.0337 0.04" rpy="1.5708 0 3.1415" />
-                <limit lower="-0.349" upper="1.5708" effort="10" velocity="3"/>
+                <limit lower="-0.349" upper="1.5708" effort="20" velocity="3"/>
                 <axis xyz="0 0 1"/>
         </joint>
