Commit message: gazebo launch fix; ros2 controller integration

File: arm_description/model/arm.urdf (robot description, URDF)
Before this commit: robot arm, 17 links, 16 joints
Links:
- added link world
- link base_link: mass None -> 1; geometry collision mesh filename=package://arm_description/model/meshes/stand/mounting_plate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 scale=0.001 0.001 0.001; visual mesh filename=package://arm_description/model/meshes/stand/mounting_plate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 scale=0.001 0.001 0.001
- link base_pulley: mass None -> 1; geometry collision mesh filename=package://arm_description/model/meshes/base/base_pulley.dae scale=0.001 0.001 0.001; visual mesh filename=package://arm_description/model/meshes/base/base_pulley.stl scale=0.001 0.001 0.001
- link base_structure: mass None -> 1; geometry collision mesh filename=package://arm_description/model/meshes/base/base_structure.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 scale=0.001 0.001 0.001; visual mesh filename=package://arm_description/model/meshes/base/base_structure.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 scale=0.001 0.001 0.001
- link base_structure_cover: mass None -> 1; geometry collision mesh filename=package://arm_description/model/meshes/base/base_structure_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 scale=0.001 0.001 0.001; visual mesh filename=package://arm_description/model/meshes/base/base_structure_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 scale=0.001 0.001 0.001
- link base_tube: mass None -> 1; geometry collision mesh filename=package://arm_description/model/meshes/stand/base_tube.dae scale=0.001 0.001 0.001; visual mesh filename=package://arm_description/model/meshes/stand/base_tube.stl scale=0.001 0.001 0.001
- link baseplate: mass None -> 1; geometry collision mesh filename=package://arm_description/model/meshes/stand/baseplate.dae scale=0.001 0.001 0.001; visual mesh filename=package://arm_description/model/meshes/stand/baseplate.stl scale=0.001 0.001 0.001
- link fore_pulley: mass None -> 1; geometry collision mesh filename=package://arm_description/model/meshes/forearm/j3_pulley.dae scale=0.001 0.001 0.001; visual mesh filename=package://arm_description/model/meshes/forearm/j3_pulley.stl scale=0.001 0.001 0.001
- link fore_rotation: mass None -> 1; geometry collision mesh filename=package://arm_description/model/meshes/forearm/forearm_rota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 scale=0.001 0.001 0.001; visual mesh filename=package://arm_description/model/meshes/forearm/forearm_rota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 scale=0.001 0.001 0.001
- link fore_structure: mass None -> 1; geometry collision mesh filename=package://arm_description/model/meshes/forearm/forearm_stru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 scale=0.001 0.001 0.001; visual mesh filename=package://arm_description/model/meshes/forearm/forearm_stru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 scale=0.001 0.001 0.001
- link j5_bearing_adapter_1: mass None -> 1; geometry collision mesh filename=package://arm_description/model/meshes/forearm/j5_bearing_a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 scale=0.001 0.001 0.001; visual mesh filename=package://arm_description/model/meshes/forearm/j5_bearing_a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 scale=0.001 0.001 0.001
- link j5_bearing_adapter_2: mass None -> 1; geometry collision mesh filename=package://arm_description/model/meshes/forearm/j5_bearing_a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 scale=0.001 0.001 0.001; visual mesh filename=package://arm_description/model/meshes/forearm/j5_bearing_a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 scale=0.001 0.001 0.001
- link j6_housing: mass None -> 1; geometry collision mesh filename=package://arm_description/model/meshes/forearm/j6_housing.d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 scale=0.001 0.001 0.001; visual mesh filename=package://arm_description/model/meshes/forearm/j6_housing.s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 scale=0.001 0.001 0.001
- link j6_nema8: mass None -> 1; geometry collision mesh filename=package://arm_description/model/meshes/forearm/j6_nema8.dae scale=0.001 0.001 0.001; visual mesh filename=package://arm_description/model/meshes/forearm/j6_nema8.stl scale=0.001 0.001 0.001
- link upper_bearing_mount: mass None -> 1; geometry collision mesh filename=package://arm_description/model/meshes/upperarm/upper_beari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 scale=0.001 0.001 0.001; visual mesh filename=package://arm_description/model/meshes/upperarm/upper_beari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 scale=0.001 0.001 0.001
- link upper_housing: mass None -> 1; geometry collision mesh filename=package://arm_description/model/meshes/upperarm/upper_housi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 scale=0.001 0.001 0.001; visual mesh filename=package://arm_description/model/meshes/upperarm/upper_housi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 scale=0.001 0.001 0.001
- link upper_pulley: mass None -> 1; geometry collision mesh filename=package://arm_description/model/meshes/upperarm/j2_pulley.d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 scale=0.001 0.001 0.001; visual mesh filename=package://arm_description/model/meshes/upperarm/j2_pulley.s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 scale=0.001 0.001 0.001
- link upper_structure: mass None -> 1; geometry collision mesh filename=package://arm_description/model/meshes/upperarm/upper_struc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 scale=0.001 0.001 0.001; visual mesh filename=package://arm_description/model/meshes/upperarm/upper_struc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 scale=0.001 0.001 0.001
Joints:
- removed joint J6
- added joint base_to_world: type fixed, parent world, child base_link, origin xyz=0 0 0 rpy=0 0 0
- added joint end_housing_nema8: type fixed, parent j6_housing, child j6_nema8, origin xyz=0 0 0.0078 rpy=0 0 0

File: arm_description/model/arm.urdf.xacro (robot description, xacro)
@@ -1,7 +1,13 @@
 <?xml version="1.0"?>
 <robot xmlns:xacro="https://www.ros.org/wiki/xacro" name="arm">
-        <xacro:arg name="prefix" default=""/>
-        <xacro:include filename="$(find arm_description)/model/arm.gazebo" />
-        <xacro:include filename="$(find arm_description)/control/control_gazebo.xacro" />
+        <xacro:include filename="$(find arm_description)/model/arm.gazebo.xacro" />
+        <xacro:include filename="$(find arm_description)/control/arm_ros2_control.xacro" />
+        <xacro:arg name="add_world" default="true"/>
+        <xacro:arg name="base_link" default="base_link"/>
+        <xacro:arg name="base_type" default="g_shape"/>
+        <xacro:arg name="flange_link" default="base_link"/>
+        <xacro:arg name="use_camera" default="false"/>
+        <xacro:arg name="use_gazebo" default="false"/>
+        <xacro:arg name="use_gripper" default="true"/>
         <material name="white">
                 <color rgba="1 1 1 1" />
@@ -14,16 +20,8 @@
         </material>
         <link name="world"/>
-        <joint name="fix_world" type="fixed">
-                <parent link="world"/>
-                <child link="base_footprint"/>
-                <origin xyz="0 0 0"/>
-        </joint>
-        <!--LINKS-->
-        <link name="base_footprint">
-        </link>
-        <joint name="base_footprint_link" type="fixed">
-                <parent link="base_footprint"/>
-                <child link="base_link"/>
-                <origin xyz="0 0 0"/>
+        <joint name="base_to_world" type="fixed">
+                <child link="base_link" />
+                <parent link="world" />
+                <origin xyz="0 0 0" rpy="0 0 0" />
         </joint>
         <!--stand-->
@@ -32,6 +30,4 @@
                         <geometry>
                                 <mesh filename="package://arm_description/model/meshes/stand/mounting_plate.stl" scale ="0.001 0.001 0.001"/>
-                        <origin xyz="0.06 -0.06 0" rpy="1.5708 0 3.1415" />
-                        <material name="white" />
                         </geometry>
                         <origin xyz="0.06 -0.06 0" rpy="1.5708 0 3.1415" />
@@ -491,6 +487,37 @@
                 <origin xyz="0 0 0.0078" rpy="0 0 0" />
         </joint>
-        <!--GAZEBO-->
-        <xacro:robot_ros2_control/>
         <xacro:arm_gazebo/>
+        <xacro:arm_ros2_control/>
+        <!--include relevant to gazebo simulation-->
+        <!--<gazebo>-->
+        <!--        <plugin-->
+        <!--                filename="gz_ros2_control-system"-->
+        <!--                name="gz_ros2_control::GazeboSimROS2ControlPlugin">-->
+        <!--                <parameters>$(find arm_simulation)/config/control_bridge.yaml</parameters>-->
+        <!--        </plugin>-->
+        <!--        <plugin-->
+        <!--                filename="gz-sim-joint-state-publisher-system"-->
+        <!--                name="gz::sim::systems::JointStatePublisher">-->
+        <!--        </plugin>-->
+        <!--        <plugin>-->
+        <!--                filename="gz-sim-pose-publisher-system"-->
+        <!--                name="gz::sim::systems::PosePublisher">-->
+        <!--                <publish_link_pose>true</publish_link_pose>-->
+        <!--                <use_pose_vector_msg>true</use_pose_vector_msg>-->
+        <!--                <publish_nested_model_pose>true</publish_nested_model_pose>-->
+        <!--        </plugin>-->
+        <!---->
+        <!--        <plugin filename="ignition-gazebo-sensors-system" name="ignition::gazebo::systems::Sensors">-->
+        <!--                <render_engine>ogre2</render_engine>-->
+        <!--        </plugin>-->
+        <!--</gazebo>-->
+        <!--<xacro:include filename="$(find arm_description)/control/gazebo_sim_ros2_control.urdf.xacro" />-->
+        <!--<xacro:load_gazebo_sim_ros2_control_plugin-->
+        <!--        use_gazebo="$(arg use_gazebo)"/>-->
+        <!---->
+        <!--<xacro:include filename="$(find arm_description)/control/arm_ros2_control.urdf.xacro" />-->
+        <!--<xacro:arm_ros2_control-->
+        <!--        flange_link="$(arg flange_link)"-->
+        <!--        use_gazebo="$(arg use_gazebo)"/>-->
+        <!---->
 </robot>

Commit message: moveit integration

File: arm_description/model/arm.urdf (robot description, URDF)
Before this commit: robot arm, 9 links, 8 joints
Joints:
- joint J1: limit lower=-3.1415 upper=3.1415 effort=1 velocity=1 -> lower=-3.1415 upper=3.1415 effort=1 velocity=10
- joint JLeft: limit lower=0 upper=0 effort=0 velocity=0 -> lower=0 upper=0.025 effort=0 velocity=10
- joint JRight: limit lower=0 upper=0 effort=0 velocity=0 -> lower=0 upper=0.025 effort=0 velocity=10

Commit message: moveit config files

File: arm_description/model/arm.urdf (robot description, URDF)
Before this commit: robot arm, 9 links, 8 joints
Joints:
- joint JLeft: limit lower=0 upper=0.025 effort=0 velocity=10 -> lower=-0.005 upper=0.031 effort=0 velocity=10
- joint JRight: limit lower=0 upper=0.025 effort=0 velocity=10 -> lower=-0.005 upper=0.031 effort=0 velocity=10

File: arm_description/model/arm.urdf.xacro (robot description, xacro)
@@ -417,6 +417,6 @@
       xyz="1 0 0" />
     <limit
-      lower="0"
-      upper="0.025"
+      lower="0.001"
+      upper="0.0251"
       effort="10"
       velocity="0.1" />
@@ -473,6 +473,6 @@
       xyz="1 0 0" />
     <limit
-      lower="0"
-      upper="0.025"
+      lower="0.001"
+      upper="0.0251"
       effort="10"
       velocity="0.1" />
